File: focesc/pcb/focesc.kicad_sch (KiCad schematic)
At the start: 0 parts

Commit message: focesc: drv8305.symbol
Parts:
- added C? (x3): 1000pf, symbol Device:C
- added C? (x4): 1uf, symbol Device:C
- added C?: 2.2uf, symbol Device:C
- added C? (x2): 47nf, symbol Device:C
- added C?: 4.7uf, symbol Device:C
- added D?: LED, symbol Device:LED
- added R?: 330, symbol Device:R
- added R?: 100, symbol Device:R
- added R? (x2): 10k, symbol Device:R
- added U?: drv8305, symbol drv8305:drv8305
Connections:
- new net: D?.1 (K), R?.1
- new net: C?.1, U?.22 (SP2)
- new net: C?.2, U?.21 (SN2)
- new net: C?.1, U?.20 (SP3)
- new net: C?.2, U?.19 (SN3)
- new net: C?.2, U?.46 (DVDD)
- new net: C?.2, U?.38 (VCP_H)
- new net: R?.1, U?.13 (PWRGD)
- new net: C?.1, U?.15 (AVDD)
- new net: C?.2, U?.23 (SN1)
- new net: C?.1, U?.24 (SP1)
- new net: C?.2, U?.37 (VCP_LSD)
- new net: C?.2, U?.39 (CP2_H)
- new net: C?.1, U?.40 (CP2_L)
- new net: C?.2, U?.41 (PVDD)
- new net: C?.1, U?.42 (CP1_L)
- new net: C?.2, U?.43 (CP1_H)
- new net: R?.1, U?.44 (VDRAIN)
- new net +3V3: C?.2, D?.2 (A), R?.1, R?.2, U?.48 (VREF)
- new net GND: C?.1, C?.1, C?.1, C?.2, U?.14 (GND), U?.45 (GND), U?.49 (PAD)
- new net PVDD: C?.1, R?.2
- new net nFAULT: C?.1, R?.2, R?.2, U?.8 (FAULT)
