File: robotvehicle/120x120/kicad/audio/audio.kicad_pcb (KiCad board)
At the start: 2 copper layers, 40.6 x 30.5 mm, 0 parts

Commit message: recent changes
Routing:
- net (no net): track 229.9 -> 263.0 mm, vias 28 -> 75
Other:
- board size 40.6 x 30.5 mm -> 50.8 x 35.6 mm
- board text added: "330k"
- board text added: "fsclk"
- board text added: "l"
- board text added: "l/r"
- board text added: "r"
