File: robotvehicle/120x120/kicad/powerswitch/vehicle.kicad_pcb (KiCad board)
At the start: 2 copper layers, 33 x 33 mm, 0 parts

Commit message: recent changes
Routing:
- net (no net): track 162.8 -> 297.2 mm
Other:
- board text added: "front"
