File: robotarthropod/6leg/pcb/6leg.kicad_pcb (KiCad board)
At the start: 2 copper layers, 77.5 x 62.2 mm, 0 parts

Commit message: simple 6leg robot(cheap 9g servo version)
Routing:
- net (no net): track 151.6 -> 168.6 mm, vias 114 -> 112
Other:
- board size 77.5 x 62.2 mm -> 71.1 x 55.9 mm
- board text removed: "0v"
- board text removed: "d"
- board text removed: "g"
- board text removed: "s"
