File: keyboard/kicad/kbd5x5.kicad_sch (KiCad schematic)
At the start: 50 parts, among them SW1 mykbd, SW10 mykbd, SW11 mykbd, SW12 mykbd, SW13 mykbd, SW14 mykbd, SW15 mykbd, SW16 mykbd, SW17 mykbd, SW18 mykbd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

Commit message: keyboard: pinout align with 2.54mm Perforated circuit board
Connections:
- net at D16.2 (DOUT), SW16.4: no longer D21.4 (DIN), SW21.3
- net at D16.4 (DIN), SW16.3: no longer D11.2 (DOUT), SW11.4
- net at D21.2 (DOUT), SW21.4: no longer D22.4 (DIN), SW22.4
- net at D3.4 (DIN), SW3.3: no longer D2.2 (DOUT), SW2.3
- net at D6.4 (DIN), SW6.3: no longer D1.2 (DOUT), SW1.4
- net at D6.2 (DOUT), SW6.4: no longer D11.4 (DIN), SW11.3
- net at D17.2 (DOUT), SW17.3: no longer D12.4 (DIN), SW12.4
- net at D17.4 (DIN), SW17.4: no longer D22.2 (DOUT), SW22.3
- net at D9.2 (DOUT), SW9.3: no longer D4.4 (DIN), SW4.4
- net at D9.4 (DIN), SW9.4: no longer D14.2 (DOUT), SW14.3
- net at D12.2 (DOUT), SW12.3: no longer D7.4 (DIN), SW7.4
- net at D5.2 (DOUT), SW5.4: no longer D10.4 (DIN), SW10.3
- net at D5.4 (DIN), SW5.3: no longer D4.2 (DOUT), SW4.3
- net at D24.2 (DOUT), SW24.3: no longer D19.4 (DIN), SW19.4
- net at D24.4 (DIN), SW24.4: no longer D23.2 (DOUT), SW23.4
- net at D7.2 (DOUT), SW7.3: no longer D2.4 (DIN), SW2.4
- net at D10.2 (DOUT), SW10.4: no longer D15.4 (DIN), SW15.3
- net at D19.2 (DOUT), SW19.3: no longer D14.4 (DIN), SW14.4
- net at D20.4 (DIN), SW20.3: no longer D15.2 (DOUT), SW15.4
- net at D20.2 (DOUT), SW20.4: no longer D25.4 (DIN), SW25.3
- new net: D21.4 (DIN), SW21.3
- new net: D22.2 (DOUT), SW22.3
- new net: D22.4 (DIN), SW22.4
- new net: D11.2 (DOUT), SW11.4
- new net: D11.4 (DIN), SW11.3
- new net: D12.4 (DIN), SW12.4
- new net: D7.4 (DIN), SW7.4
- new net: D10.4 (DIN), SW10.3
- new net: D23.2 (DOUT), SW23.4
- new net: D19.4 (DIN), SW19.4
- new net: D4.2 (DOUT), SW4.3
- new net: D4.4 (DIN), SW4.4
- new net: D25.4 (DIN), SW25.3
- new net: D2.2 (DOUT), SW2.3
- new net: D2.4 (DIN), SW2.4
- new net: D15.4 (DIN), SW15.3
- new net: D15.2 (DOUT), SW15.4
- new net: D14.2 (DOUT), SW14.3
- new net: D14.4 (DIN), SW14.4
- new net: D1.2 (DOUT), SW1.4

Commit message: keyboard pcb: bottom board(esp32s3 minimal 20mmx40mm)
Connections:
- net at D3.2 (DOUT), SW3.4: no longer D8.4 (DIN), SW8.3
- net at D13.4 (DIN), SW13.3: no longer D8.2 (DOUT), SW8.4
- net at D13.2 (DOUT), SW13.4: no longer D18.4 (DIN), SW18.3
- net at D23.4 (DIN), SW23.3: no longer D18.2 (DOUT), SW18.4
- new net: D18.2 (DOUT), SW18.4
- new net: D18.4 (DIN), SW18.3
- new net: D8.4 (DIN), SW8.3
- new net: D8.2 (DOUT), SW8.4
