File: input/keyboard/kicad/kbd2x2.kicad_pcb (KiCad board)
At the start: 2 copper layers, 40 x 40 mm, 8 parts, among them SW1 mykbd, SW2 mykbd, SW3 mykbd, SW4 mykbd

Commit message: reorganize dir, keyboard pcb update
Parts:
- removed D3, D4: WS2812B, LED_SMD:LED_WS2812B_PLCC4_5.0x5.0mm_P3.2mm
- SW4: footprint mykbd:seat -> mykbd:seat_b
Connections:
- SW3 pad 3: Net-(D3-DIN) -> unconnected-(SW3-Pad3)
- SW3 pad 4: Net-(D3-DOUT) -> unconnected-(SW3-Pad4)
- SW4 pad 3: Net-(D4-DOUT) -> unconnected-(SW4-Pad3)
- SW4 pad 4: Net-(D4-DIN) -> unconnected-(SW4-Pad4)
Routing:
- net GND: track 340.5 -> 254.3 mm, vias 0 -> 2
- net VCC: track 249.0 -> 222.4 mm
- net Net-(D3-DOUT): track 24.4 -> 0.00 mm
- net unconnected-(SW3-Pad4): track 0.00 -> 23.1 mm
- net Net-(D4-DOUT): track 22.5 -> 0.00 mm, vias 1 -> 0
- net unconnected-(SW4-Pad4): track 0.00 -> 21.6 mm, vias 0 -> 1
- net Net-(D4-DIN): track 20.0 -> 0.00 mm
- net unconnected-(SW3-Pad3): track 0.00 -> 19.8 mm, vias 0 -> 1
- net unconnected-(SW4-Pad3): track 0.00 -> 19.7 mm
- net Net-(D3-DIN): track 19.5 -> 0.00 mm, vias 1 -> 0
- net Net-(SW3-Pad2): track 46.4 -> 39.4 mm
- net Net-(SW1-Pad1): track 47.0 -> 44.0 mm
- net Net-(SW2-Pad1): track 47.0 -> 44.5 mm
Other:
- board text added: "ws2812b-32x28"
