File: input/keyboard/kicad/esp32s3-wroom1/esp32s3-wroom1.kicad_pcb (KiCad board)
At the start: 2 copper layers, 40 x 80 mm, 31 parts, among them J1 Conn_01x01_Pin, J10 Conn_01x01_Pin, J11 USB_C_Receptacle_USB2.0_16P, J12 Conn_01x02_Pin, J13 Conn_01x16_Pin, J14 Conn_01x04_Pin, J2 Conn_01x01_Pin, J3 Conn_01x01_Pin, J4 Conn_01x01_Pin, J5 Conn_01x02_Pin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

Commit message: input/keyboard: newest working version
Connections:
- net y4 renamed g15
- net y5 renamed g16
- net y6 renamed g17
- net y7 renamed g18
Routing:
- net g3: track 98.7 -> 58.3 mm, vias 2 -> 1
- net GND: track 243.7 -> 268.1 mm, vias 17 -> 19
- net x1: track 37.3 -> 57.7 mm, vias 3 -> 5
- net g15: track 18.1 -> 37.7 mm, vias 1 -> 2
- net x0: track 71.1 -> 85.1 mm, vias 2 -> 3
- net g46: track 67.9 -> 61.3 mm, vias 2 -> 1
- net g0: track 53.3 -> 50.8 mm, vias 2 -> 1
- net Net-(J5-Pin_2): track 55.9 -> 53.4 mm
- net Net-(J5-Pin_1): track 54.8 -> 52.6 mm
- net g45: track 49.6 -> 47.7 mm
- net y3: track 63.5 -> 62.0 mm
- net y1: track 26.1 -> 24.8 mm
- net +5V: track 157.2 -> 158.0 mm
- net g18: track 21.5 -> 22.3 mm
- net g17: track 20.5 -> 21.3 mm
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Other:
- outline, holes or cut-outs redrawn
- board text added: "0,boot"
- board text added: "0.1uf"
- board text added: "10uf"
- board text removed: "boot"
